File: mseq.kicad_sch (KiCad schematic)
At the start: 87 parts, among them J1 Screen_I2C, J3 Conn_ARM_JTAG_SWD_10, SW1 RESET, SW2 ON/OFF, SW3 MS/SLAVE, SW4 BOOT, U1 SN74HCT125DR, U2 H11L1M, U3 AMS1117-3.3, U4 STM32F413CHUx, U5 CP2102N-Axx-xQFN20, U6 H11L1M, U7 W25Q16JVSS, U8 MB85RS256B, Y1 32.768kHz ±20ppm 6pF, Y2 25 MHz ±20ppm 18pF

Commit message: chaged the pin name
Connections:
- net B6 renamed SCL
- net B7 renamed SDA
Changed lines of the file:
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@@
 		)
 	)
-	(label "B7"
+	(label "SDA"
 		(at 349.25 25.4 0)
 		(effects
@@
 		)
 	)
-	(label "B6"
+	(label "SCL"
 		(at 257.81 130.81 0)
 		(effects
@@
 		)
 	)
-	(label "B6"
+	(label "SCL"
 		(at 349.25 22.86 0)
 		(effects
@@
 		)
 	)
-	(label "B7"
+	(label "SDA"
 		(at 257.81 133.35 0)
 		(effects

Commit message: updated
Connections:
- net +3.3V: now also J1.2 (Pin_2); no longer J1.3 (Pin_3)
- net GND: now also J1.1 (Pin_1); no longer J1.4 (Pin_4)
- net SCL: now also J1.3 (Pin_3); no longer J1.1 (Pin_1)
- net SDA: now also J1.4 (Pin_4); no longer J1.2 (Pin_2)
Changed lines of the file:
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@@
 		(exclude_from_sim no)
 		(at 334.01 13.97 0)
-		(size 26.67 26.67)
+		(size 24.13 26.67)
 		(margins 0.9525 0.9525 0.9525 0.9525)
 		(stroke
@@
 	(wire
 		(pts
-			(xy 345.44 25.4) (xy 349.25 25.4)
-		)
-		(stroke
-			(width 0)
-			(type default)
-		)
-	)
-	(wire
-		(pts
 			(xy 256.54 148.59) (xy 265.43 148.59)
 		)
@@
 	(wire
 		(pts
-			(xy 345.44 22.86) (xy 349.25 22.86)
-		)
-		(stroke
-			(width 0)
-			(type default)
-		)
-	)
-	(wire
-		(pts
 			(xy 149.86 265.43) (xy 152.4 265.43)
 		)
@@
 	(wire
 		(pts
-			(xy 345.44 27.94) (xy 356.87 27.94)
+			(xy 345.44 27.94) (xy 349.25 27.94)
 		)
 		(stroke
@@
 	(wire
 		(pts
-			(xy 356.87 30.48) (xy 356.87 33.02)
-		)
-		(stroke
-			(width 0)
-			(type default)
-		)
-	)
-	(wire
-		(pts
 			(xy 255.27 262.89) (xy 255.27 266.7)
 		)
@@
 	(wire
 		(pts
-			(xy 345.44 30.48) (xy 356.87 30.48)
+			(xy 46.99 245.11) (xy 66.04 245.11)
 		)
 		(stroke
@@
 	(wire
 		(pts
-			(xy 46.99 245.11) (xy 66.04 245.11)
+			(xy 63.5 226.06) (xy 63.5 261.62)
 		)
 		(stroke
@@
 	(wire
 		(pts
-			(xy 63.5 226.06) (xy 63.5 261.62)
+			(xy 113.03 44.45) (xy 113.03 46.99)
 		)
 		(stroke
@@
 	(wire
 		(pts
-			(xy 113.03 44.45) (xy 113.03 46.99)
+			(xy 16.51 146.05) (xy 21.59 146.05)
 		)
 		(stroke
@@
 	(wire
 		(pts
-			(xy 16.51 146.05) (xy 21.59 146.05)
+			(xy 345.44 30.48) (xy 349.25 30.48)
 		)
 		(stroke
@@
 	(wire
 		(pts
+			(xy 345.44 21.59) (xy 349.25 21.59)
+		)
+		(stroke
+			(width 0)
+			(type default)
+		)
+	)
+	(wire
+		(pts
 			(xy 401.32 170.18) (xy 401.32 175.26)
 		)
@@
 	(wire
 		(pts
-			(xy 356.87 25.4) (xy 356.87 27.94)
+			(xy 353.06 24.13) (xy 353.06 25.4)
 		)
 		(stroke
@@
 	(wire
 		(pts
+			(xy 345.44 25.4) (xy 353.06 25.4)
+		)
+		(stroke
+			(width 0)
+			(type default)
+		)
+	)
+	(wire
+		(pts
 			(xy 172.72 222.25) (xy 170.18 222.25)
 		)
@@
 	(wire
 		(pts
+			(xy 345.44 21.59) (xy 345.44 22.86)
+		)
+		(stroke
+			(width 0)
+			(type default)
+		)
+	)
+	(wire
+		(pts
 			(xy 69.85 41.91) (xy 69.85 44.45)
 		)
@@
 	)
 	(label "SDA"
-		(at 349.25 25.4 0)
+		(at 349.25 30.48 0)
 		(effects
 			(font
@@
 	)
 	(label "SCL"
-		(at 349.25 22.86 0)
+		(at 349.25 27.94 0)
 		(effects
 			(font
@@
 	(symbol
 		(lib_id "power:+3.3V")
-		(at 356.87 25.4 0)
+		(at 353.06 24.13 0)
 		(unit 1)
 		(body_style 1)
@@
 		(dnp no)
 		(property "Reference" "#PWR037"
-			(at 356.87 29.21 0)
+			(at 353.06 27.94 0)
 			(hide yes)
 			(show_name no)
@@
 		)
 		(property "Value" "+3.3V"
-			(at 356.616 21.336 0)
+			(at 352.806 20.066 0)
 			(show_name no)
 			(do_not_autoplace no)
@@
 		)
 		(property "Footprint" ""
-			(at 356.87 25.4 0)
+			(at 353.06 24.13 0)
 			(hide yes)
 			(show_name no)
@@
 		)
 		(property "Datasheet" ""
-			(at 356.87 25.4 0)
+			(at 353.06 24.13 0)
 			(hide yes)
 			(show_name no)
@@
 		)
 		(property "Description" "Power symbol creates a global label with name \"+3.3V\""
-			(at 356.87 25.4 0)
+			(at 353.06 24.13 0)
 			(hide yes)
 			(show_name no)
@@
 	(symbol
 		(lib_id "power:GND")
-		(at 356.87 33.02 0)
+		(at 349.25 21.59 0)
 		(unit 1)
 		(body_style 1)
@@
 		(fields_autoplaced yes)
 		(property "Reference" "#PWR038"
-			(at 356.87 39.37 0)
+			(at 349.25 27.94 0)
 			(hide yes)
 			(show_name no)
@@
 		)
 		(property "Value" "GND"
-			(at 356.87 38.1 0)
+			(at 349.25 26.67 0)
 			(hide yes)
 			(show_name no)
@@
 		)
 		(property "Footprint" ""
-			(at 356.87 33.02 0)
+			(at 349.25 21.59 0)
 			(hide yes)
 			(show_name no)
@@
 		)
 		(property "Datasheet" ""
-			(at 356.87 33.02 0)
+			(at 349.25 21.59 0)
 			(hide yes)
 			(show_name no)
@@
 		)
 		(property "Description" "Power symbol creates a global label with name \"GND\" , ground"
-			(at 356.87 33.02 0)
+			(at 349.25 21.59 0)
 			(hide yes)
 			(show_name no)
