File: mseq.kicad_pcb (KiCad board)
At the start: 2 copper layers, 100 x 67 mm, 87 parts, among them J1 Screen_I2C, J3 Conn_ARM_JTAG_SWD_10, SW1 RESET, SW2 ON/OFF, SW3 MS/SLAVE, SW4 BOOT, U1 SN74HCT125DR, U2 H11L1M, U3 AMS1117-3.3, U4 STM32F413CHUx, U5 CP2102N-Axx-xQFN20, U6 H11L1M, U7 W25Q16JVSS, U8 MB85RS256B, Y1 32.768kHz ±20ppm 6pF, Y2 25 MHz ±20ppm 18pF

Commit message: PCB updated, wip
Parts:
- moved R17 72.8 mm to (135.7, 60.9), turned to 180 degrees
- moved D2 69.2 mm to (141.6, 63.0)
- moved R18 63.6 mm to (147.0, 60.9)
- moved FB1 13.2 mm to (70.5, 69.7)
- moved FB2 13.2 mm to (79.8, 69.8)
- moved R3 13.2 mm to (73.5, 69.7)
- moved MIDI_IN1 13.2 mm to (74.8, 55.9)
- moved FB4 9.40 mm to (92.5, 69.3)
- moved FB7 9.40 mm to (103.9, 69.6)
- moved MIDI_OUT1 9.40 mm to (98.2, 55.9)
- moved R4 9.40 mm to (89.5, 69.3)
- moved R8 9.40 mm to (107.1, 69.6)
- moved FB3 5.10 mm to (115.7, 69.8)
- moved MIDI_THRU1 5.10 mm to (121.4, 55.9)
- moved R2 5.10 mm to (112.7, 69.8)
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Routing:
- net GND: track 554.2 -> 489.2 mm, vias 116 -> 117
- net Net-(USB1-CC1): track 0.00 -> 14.6 mm, vias 0 -> 3
- net Net-(USB1-CC2): track 0.00 -> 12.6 mm, vias 0 -> 2
- net /D-: track 36.7 -> 47.6 mm, vias 0 -> 4
- net (no net): track 10.00 -> 0.00 mm
- net /D+: track 36.0 -> 44.2 mm
- net Net-(SW2-B): track 22.2 -> 23.9 mm
- net VBUS: track 93.2 -> 94.8 mm
- net +3.3V: track 270.2 -> 270.8 mm
Other:
- board size 100 x 67 mm -> 101.3 x 67.6 mm

Commit message: PCB placement & routing WIP
Parts:
- added REF**: MountingHole_3.2mm_M3, MountingHole:MountingHole_3.2mm_M3, F.Cu at (40.0, 111.5)
- moved R12 141.0 mm to (66.6, 69.5)
- moved FB8 139.9 mm to (70.0, 69.2), turned to 180 degrees
- moved FB9 130.9 mm to (78.8, 69.3)
- moved R19 129.4 mm to (72.9, 69.3), turned to 180 degrees
- moved U6 127.9 mm to (78.1, 74.3)
- moved D7 127.7 mm to (84.4, 69.3), turned to 180 degrees
- moved D6 121.4 mm to (70.7, 73.9), turned to -90 degrees
- moved C22 119.5 mm to (85.1, 72.8), turned to -90 degrees
- moved R21 117.4 mm to (89.5, 69.5)
- moved R20 114.7 mm to (87.9, 72.8), turned to 90 degrees
- moved MIDI_IN2 111.2 mm to (74.9, 55.9), turned to -90 degrees
- moved FB2 24.8 mm to (55.0, 69.2)
- moved FB1 23.5 mm to (47.0, 69.2)
- moved MIDI_IN1 23.4 mm to (51.4, 55.9)
- moved R3 23.4 mm to (50.1, 69.3)
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Routing:
- net GND: track 489.2 -> 424.0 mm, vias 117 -> 121
- net +3.3V: track 270.8 -> 214.5 mm, vias 7 -> 9
- net /B3: track 66.5 -> 28.2 mm
- net /A15: track 78.0 -> 44.2 mm, vias 2 -> 1
- net /A3: track 0.00 -> 16.3 mm, vias 0 -> 2
- net Net-(R4-Pad2): track 29.9 -> 16.3 mm
- net Net-(D6-A): track 0.00 -> 12.4 mm
- net Net-(D7-A): track 0.00 -> 11.6 mm, vias 0 -> 2
- net Net-(D4-A): track 3.13 -> 12.2 mm, vias 0 -> 2
- net Net-(FB9-Pad2): track 0.00 -> 6.07 mm
- net Net-(FB8-Pad2): track 0.00 -> 6.05 mm
- net Net-(D6-K): track 0.00 -> 5.47 mm
- net Net-(FB7-Pad2): track 6.21 -> 11.6 mm
- net Net-(FB4-Pad1): track 5.92 -> 0.55 mm
- net Net-(FB8-Pad1): track 0.00 -> 1.44 mm
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Other:
- board size 101.3 x 67.6 mm -> 113.7 x 67.6 mm
- board text added: "MSeq v1.0.0"
- board text removed: "MIDI IN"
- board text removed: "MSeq v0.1.0"

Commit message: PCB placement & routing WIP
Parts:
- moved J3 103.4 mm to (99.8, 111.2), turned to 90 degrees
- moved C23 92.6 mm to (125.6, 99.9)
- moved U8 90.1 mm to (118.6, 105.0)
- moved U7 89.5 mm to (118.5, 98.6)
- moved C7 12.5 mm to (96.7, 88.3), turned to 90 degrees
- moved C12 2.83 mm to (99.8, 87.9), turned to 90 degrees
- moved FB6 2.57 mm to (92.0, 98.8), turned to -90 degrees
- moved C19 2.20 mm to (103.8, 100.3)
- moved R9 1.80 mm to (100.6, 85.6)
- moved C2 1.71 mm to (104.0, 98.5)
- moved C8 1.59 mm to (93.8, 98.2), turned to -90 degrees
- moved C11 1.44 mm to (95.5, 98.0), turned to -90 degrees
- moved SW4 1.40 mm to (146.7, 109.7)
- moved C4 1.30 mm to (106.2, 90.5)
- moved C5 0.73 mm to (98.2, 87.9), turned to 90 degrees
Routing:
- net /NRST: track 99.4 -> 55.5 mm
- net +3.3V: track 214.5 -> 171.4 mm, vias 9 -> 8
- net /B6: track 48.8 -> 11.4 mm
- net /SWCLOCK: track 26.8 -> 0.00 mm, vias 2 -> 0
- net /SWDIO: track 25.4 -> 0.00 mm, vias 2 -> 0
- net GND: track 424.0 -> 402.0 mm, vias 121 -> 125
- net /B7: track 49.1 -> 32.5 mm, vias 2 -> 1
- net VDDA: track 9.96 -> 7.27 mm
- net Net-(U4-VCAP_1): track 5.84 -> 3.40 mm
- net /BOOT0: track 61.3 -> 62.8 mm
