File: mseq.kicad_pcb (KiCad board)
At the start: 2 copper layers, 135.3 x 78.4 mm, 93 parts, among them J1 Screen_I2C, J3 Conn_ARM_JTAG_SWD_10, SW1 RESET, SW2 ON/OFF, SW3 MS/SLAVE, SW4 BOOT, U1 SN74HCT125DR, U2 H11L1M, U3 AMS1117-3.3, U4 STM32F413CHUx, U5 CP2102N-Axx-xQFN20, U6 H11L1M, U7 W25Q16JVSS, U8 MB85RS256B, Y1 32.768kHz ±20ppm 6pF, Y2 25 MHz ±20ppm 18pF

Commit message: Vias added
Routing:
- net GND: track 422.5 -> 428.5 mm, vias 130 -> 134
Changed lines of the file:
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@@
 	)
 	(segment
+		(start 95.55 101.09)
+		(end 95.06 101.58)
+		(width 0.4)
+		(layer "F.Cu")
+		(net "GND")
+	)
+	(segment
 		(start 89.3 97.55)
 		(end 89.732844 97.55)
@@
 	)
 	(segment
+		(start 95.55 98.75)
+		(end 95.55 101.09)
+		(width 0.4)
+		(layer "F.Cu")
+		(net "GND")
+	)
+	(segment
 		(start 132.275 71.8)
 		(end 132.975 72.5)
@@
 	)
 	(segment
+		(start 93.75 99.15)
+		(end 93.75 100.27)
+		(width 0.4)
+		(layer "F.Cu")
+		(net "GND")
+	)
+	(segment
 		(start 105.3 101.7)
 		(end 105.3 100.35)
@@
 	)
 	(segment
+		(start 93.75 100.27)
+		(end 95.06 101.58)
+		(width 0.4)
+		(layer "F.Cu")
+		(net "GND")
+	)
+	(segment
 		(start 129.875 86.625)
 		(end 129.875 87.4)
@@
 	)
 	(via
-		(at 101.4 58.3)
+		(at 97.75 53.65)
 		(size 0.7)
 		(drill 0.3)
@@
 	)
 	(via
+		(at 130.08 81.64)
+		(size 0.7)
+		(drill 0.3)
+		(layers "F.Cu" "B.Cu")
+		(free yes)
+		(capping no)
+		(covering
+			(front no)
+			(back no)
+		)
+		(plugging
+			(front no)
+			(back no)
+		)
+		(filling no)
+		(net "GND")
+	)
+	(via
 		(at 68.75 75.3)
 		(size 0.7)
@@
 	)
 	(via
-		(at 125.5 58.8975)
+		(at 115.5 57.1)
 		(size 0.7)
 		(drill 0.3)
@@
 	)
 	(via
+		(at 91.74 96.03)
+		(size 0.7)
+		(drill 0.3)
+		(layers "F.Cu" "B.Cu")
+		(net "GND")
+	)
+	(via
 		(at 54.8 58.6)
 		(size 0.7)
@@
 	)
 	(via
-		(at 102.9 60.5)
+		(at 104.05 55.55)
 		(size 0.7)
 		(drill 0.3)
@@
 	)
 	(via
+		(at 95.06 101.58)
+		(size 0.7)
+		(drill 0.3)
+		(layers "F.Cu" "B.Cu")
+		(free yes)
+		(capping no)
+		(covering
+			(front no)
+			(back no)
+		)
+		(plugging
+			(front no)
+			(back no)
+		)
+		(filling no)
+		(net "GND")
+	)
+	(via
 		(at 35.85 80.85)
 		(size 0.7)
@@
 	)
 	(via
+		(at 39.85 104.1)
+		(size 0.7)
+		(drill 0.3)
+		(layers "F.Cu" "B.Cu")
+		(free yes)
+		(capping no)
+		(covering
+			(front no)
+			(back no)
+		)
+		(plugging
+			(front no)
+			(back no)
+		)
+		(filling no)
+		(net "GND")
+	)
+	(via
 		(at 137.5 85.8)
 		(size 0.7)
@@
 	)
 	(via
-		(at 118.2 58.7975)
+		(at 120.6 54.4)
 		(size 0.7)
 		(drill 0.3)
@@
 		(polygon
 			(pts
-				(xy 89.8 97.6) (xy 89.8 97) (xy 89.6 97) (xy 89.6 97.6)
+				(xy 89.91 97.98) (xy 89.91 97.18) (xy 89.6 97.18) (xy 89.6 97.98)
 			)
 		)
