File: mseq.kicad_pcb (KiCad board)
At the start: 2 copper layers, 135.3 x 78.4 mm, 93 parts, among them J1 Screen_I2C, J3 Conn_ARM_JTAG_SWD_10, SW1 RESET, SW2 ON/OFF, SW3 MS/SLAVE, SW4 BOOT, U1 SN74HCT125DR, U2 H11L1M, U3 AMS1117-3.3, U4 STM32F413CHUx, U5 CP2102N-Axx-xQFN20, U6 H11L1M, U7 W25Q16JVSS, U8 MB85RS256B, Y1 32.768kHz ±20ppm 6pF, Y2 25 MHz ±20ppm 18pF

Commit message: chaged the pin name
Connections:
- net /B6 renamed /SCL
- net /B7 renamed /SDA

Commit message: updated
Parts:
- removed the REF** at (18.2, 52.5)
- moved REF** 27.0 mm to (45.0, 80.0)
- moved REF** 27.0 mm to (45.0, 119.0)
- moved REF** 27.0 mm to (113.0, 80.0)
- moved REF** 27.0 mm to (113.0, 119.0)
- moved J3 25.2 mm to (131.9, 115.5)
- moved D3 23.1 mm to (38.5, 72.5)
- moved R11 22.3 mm to (43.2, 71.8)
- moved REF** 3.40 mm to (145.2, 119.0)
Connections:
- J1 pad 1: /SCL -> GND
- J1 pad 2: /SDA -> +3.3V
- J1 pad 3: +3.3V -> /SCL
- J1 pad 4: GND -> /SDA
Routing:
- net +3.3V: track 486.3 -> 378.9 mm
- net /SWDIO: track 31.2 -> 15.6 mm
- net GND: track 428.5 -> 414.9 mm, vias 134 -> 132
- net /NRST: track 102.6 -> 92.3 mm
- net /SWCLOCK: track 40.2 -> 36.8 mm, vias 4 -> 3
- net /SDA: track 106.7 -> 103.4 mm, vias 3 -> 4
- net Net-(D3-A): track 5.00 -> 4.39 mm
Other:
- board size 135.3 x 78.4 mm -> 113 x 74.5 mm

Commit message: Wip
Parts:
- added REF**: MountingHole_3.2mm_M3, MountingHole:MountingHole_3.2mm_M3, F.Cu at (41.0, 114.0)
- added REF**: MountingHole_3.2mm_M3, MountingHole:MountingHole_3.2mm_M3, F.Cu at (41.0, 75.0)
- added REF**: MountingHole_3.2mm_M3, MountingHole:MountingHole_3.2mm_M3, F.Cu at (149.4, 52.1)
- moved D1 14.5 mm to (56.8, 85.2)
- moved U2 14.3 mm to (64.1, 86.2)
- moved C9 14.2 mm to (71.2, 84.7)
- moved D8 13.2 mm to (135.2, 113.3)
- moved R23 13.2 mm to (140.7, 113.3)
- moved R22 13.2 mm to (132.0, 113.3)
- moved D9 13.2 mm to (143.7, 113.2)
- moved SW4 7.16 mm to (150.6, 103.7)
- moved REF** 7.07 mm to (50.0, 75.0)
- moved REF** 7.07 mm to (50.0, 114.0)
- moved REF** 7.07 mm to (118.0, 75.0)
- moved REF** 7.07 mm to (118.0, 114.0)
- moved J3 7.01 mm to (125.3, 113.2)
- moved REF** 6.72 mm to (149.4, 113.8)
- moved SW3 6.08 mm to (150.7, 92.4)
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Routing:
- net /SWDIO: track 15.6 -> 36.5 mm, vias 2 -> 4
- net /SWCLOCK: track 36.8 -> 52.4 mm, vias 3 -> 4
- net Net-(D1-K): track 5.64 -> 19.3 mm
- net Net-(D1-A): track 11.2 -> 22.3 mm
- net /BOOT0: track 62.8 -> 70.4 mm
- net +3.3V: track 378.9 -> 385.6 mm, vias 15 -> 13
- net GND: track 414.9 -> 421.5 mm, vias 132 -> 139
- net /B3: track 64.0 -> 70.6 mm, vias 4 -> 2
- net /TXT: track 49.8 -> 44.0 mm
- net Net-(SW3-A): track 6.05 -> 11.6 mm
- net /A1: track 65.0 -> 70.5 mm
- net /NRST: track 92.3 -> 97.7 mm, vias 4 -> 3
- net /RXT: track 52.2 -> 47.6 mm
- net VBUS: track 91.9 -> 95.3 mm
- net Net-(SW2-B): track 23.9 -> 25.5 mm
Other:
- board size 113 x 74.5 mm -> 116.5 x 69.6 mm
- board text added: "MSeq v1.1.0"
- board text removed: "MSeq v1.0.0"
